File: _autosave-ai03-pcb-guide.kicad_pcb (KiCad board)
At the start: 2 copper layers, 76.2 x 38.1 mm, 24 parts, among them SW1 SW_Push, U1 ATmega32U4-AU, Y1 16MHz

Commit message: Generate gerbers
Routing:
- added copper zone on B.Cu, net GND
Other:
- board text added: "Hello World!"
Changed lines of the file:
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@@
   (general
     (thickness 1.6)
-    (drawings 8)
+    (drawings 9)
     (tracks 210)
     (zones 0)
@@
     (visible_elements FFFFFF7F)
     (pcbplotparams
-      (layerselection 0x010fc_ffffffff)
-      (usegerberextensions false)
+      (layerselection 0x010f0_ffffffff)
+      (usegerberextensions true)
       (usegerberattributes false)
       (usegerberadvancedattributes false)
@@
       (plotinvisibletext false)
       (padsonsilk false)
-      (subtractmaskfromsilk false)
+      (subtractmaskfromsilk true)
       (outputformat 1)
       (mirror false)
-      (drillshape 1)
+      (drillshape 0)
       (scaleselection 1)
-      (outputdirectory ""))
+      (outputdirectory "Gerbers"))
   )
   (net 0 "")
@@
       (rotate (xyz 0 0 0))
     )
+  )
+  (gr_text "Hello World!" (at 40.48125 97.63125) (layer F.SilkS)
+    (effects (font (size 1.5 1.5) (thickness 0.3)))
   )
   (gr_arc (start 105.56875 64.29375) (end 107.95 64.29375) (angle -90) (layer Edge.Cuts) (width 0.2))
@@
   (segment (start 66.487 86.553) (end 68.199 86.553) (width 0.254) (layer B.Cu) (net 28))
   (segment (start 66.23 86.296) (end 66.487 86.553) (width 0.254) (layer B.Cu) (net 28))
+  (zone (net 2) (net_name GND) (layer B.Cu) (hatch edge 0.508)
+    (connect_pads (clearance 0.508))
+    (min_thickness 0.254)
+    (fill yes (arc_segments 16) (thermal_gap 0.508) (thermal_bridge_width 0.508))
+    (polygon
+      (pts
+        (xy 35.71875 69.05625) (xy 43.65625 69.05625) (xy 43.65625 61.9125) (xy 35.71875 61.9125)
+      )
+    )
+  )
+  (zone (net 2) (net_name GND) (layer B.Cu) (hatch edge 0.508)
+    (connect_pads (clearance 0.508))
+    (min_thickness 0.254)
+    (fill yes (arc_segments 16) (thermal_gap 0.508) (thermal_bridge_width 0.508))
+    (polygon
+      (pts
+        (xy 50.8 65.0875) (xy 66.675 65.0875) (xy 66.675 75.40625) (xy 50.8 75.40625)
+      )
+    )
+  )
+  (zone (net 2) (net_name GND) (layer B.Cu) (hatch edge 0.508)
+    (connect_pads (clearance 0.508))
+    (min_thickness 0.254)
+    (fill yes (arc_segments 16) (thermal_gap 0.508) (thermal_bridge_width 0.508))
+    (polygon
+      (pts
+        (xy 53.975 77.7875) (xy 63.5 77.7875) (xy 63.5 87.3125) (xy 53.975 87.3125)
+      )
+    )
+  )
 )
